Commit message: Set the geometry of the robot

File: description/robot_core.xacro (robot description, xacro)
@@ -1,3 +1,31 @@
 <?xml version="1.0"?>
 <robot xmlns:xacro="http://www.ros.org/wiki/xacro" >
+    <material name="white">
+        <color rgba="1 1 1 1" />
+    <material/>
+    <material name="orange">
+        <color rgba="1 0.3 0.1 1" />
+    <material/>
+    <material name="blue">
+        <color rgba="0.2 0.2 1 1" />
+    <material/>
+    <material name="black">
+        <color rgba="0 0 0 1" />
+    <material/>
+    <link name="base_link">
+    </link>
+    <joint name="chassis_joint" type="fixed">
+        <parent link="base_link" />
+        <child link="chassis"/>
+        <origin xyz="-0.1 0 0"/>
+    </joint>
+    <link name="chassis">
+        <visual>
+            <origin xyz="0.13 0 0.03"/>
+            <geometry>
+                <box size="0.26 0.2 0.06"/>
+            </geometry>
+            <material name="white"/>
+        </visual>
+    </link>
 </robot>

Commit message: Fixed syntax errors

File: description/robot_core.xacro (robot description, xacro)
@@ -1,16 +1,16 @@
 <?xml version="1.0"?>
-<robot xmlns:xacro="http://www.ros.org/wiki/xacro" >
+<robot xmlns:xacro="http://www.ros.org/wiki/xacro">
     <material name="white">
-        <color rgba="1 1 1 1" />
-    <material/>
+        <color rgba="1 1 1 1"/>
+    </material>
     <material name="orange">
         <color rgba="1 0.3 0.1 1" />
-    <material/>
+    </material>
     <material name="blue">
         <color rgba="0.2 0.2 1 1" />
-    <material/>
+    </material>
     <material name="black">
         <color rgba="0 0 0 1" />
-    <material/>
+    </material>
     <link name="base_link">
     </link>

Commit message: added left and right wheels

File: description/robot_core.xacro (robot description, xacro)
@@ -13,6 +13,8 @@
         <color rgba="0 0 0 1" />
     </material>
+    <!-- BASE LINK -->
     <link name="base_link">
     </link>
+    <!-- CHASSIS LINK -->
     <joint name="chassis_joint" type="fixed">
         <parent link="base_link" />
@@ -29,3 +31,33 @@
         </visual>
     </link>
+    <!-- LEFT WHEEL LINK-->
+    <joint name="left_wheel_joint" type="continuous">
+        <parent link="base_link" />
+        <child link="left_wheel"/>
+        <origin xyz="0 0.175 0" rpy="-${pi/2} 0 0"/>
+        <axis xyz="0 0 1"/>
+    </joint>
+    <link name="left_wheel">
+        <visual>
+            <geometry>
+                <cylinder radius="0.05" length="0.04"/>
+            </geometry>
+            <material name="blue"/>
+        </visual>
+    </link>
+    <!-- RIGHT WHEEL LINK-->
+    <joint name="right_wheel_joint" type="continuous">
+        <parent link="base_link" />
+        <child link="right_wheel"/>
+        <origin xyz="0 -0.175 0" rpy="${pi/2} 0 0"/>
+        <axis xyz="0 0 -1"/>
+    </joint>
+    <link name="right_wheel">
+        <visual>
+            <geometry>
+                <cylinder radius="0.05" length="0.04"/>
+            </geometry>
+            <material name="blue"/>
+        </visual>
+    </link>
 </robot>

Commit message: created caster wheel (change to front wheels l8r)

File: description/robot_core.xacro (robot description, xacro)
@@ -61,3 +61,17 @@
         </visual>
     </link>
+    <!-- FRONT WHEEL LINK-->
+    <joint name="front_wheel_joint" type="fixed">
+        <parent link="chassis"/>
+        <child link="front_wheel"/>
+        <origin xyz="0.24 0 0"/>
+    </joint>
+    <link name="caster_wheel">
+        <visual>
+            <geometry>
+                <sphere radius="0.05"/>
+            </geometry>
+            <material name="black"/>
+        </visual>
+    </link>
 </robot>

Commit message: corrected syntax errors

File: description/robot_core.xacro (robot description, xacro)
@@ -67,5 +67,5 @@
         <origin xyz="0.24 0 0"/>
     </joint>
-    <link name="caster_wheel">
+    <link name="front_wheel">
         <visual>
             <geometry>

Commit message: added collision tags to joints

File: description/robot_core.xacro (robot description, xacro)
@@ -30,4 +30,10 @@
             <material name="white"/>
         </visual>
+        <collision>
+            <origin xyz="0.13 0 0.03"/>
+            <geometry>
+                <box size="0.26 0.2 0.06"/>
+            </geometry>
+        </collision>
     </link>
     <!-- LEFT WHEEL LINK-->
@@ -45,4 +51,9 @@
             <material name="blue"/>
         </visual>
+        <collision>
+            <geometry>
+                <cylinder radius="0.05" length="0.04"/>
+            </geometry>
+        </collision>
     </link>
     <!-- RIGHT WHEEL LINK-->
@@ -60,4 +71,9 @@
             <material name="blue"/>
         </visual>
+        <collision>
+            <geometry>
+                <cylinder radius="0.05" length="0.04"/>
+            </geometry>
+        </collision>
     </link>
     <!-- FRONT WHEEL LINK-->
@@ -74,4 +90,9 @@
             <material name="black"/>
         </visual>
+        <collision>
+            <geometry>
+                <sphere radius="0.05"/>
+            </geometry>
+        </collision>
     </link>
 </robot>

Commit message: created interia macros and tags for components

File: description/robot_core.xacro (robot description, xacro)
@@ -1,4 +1,5 @@
 <?xml version="1.0"?>
 <robot xmlns:xacro="http://www.ros.org/wiki/xacro">
+    <xacro:include filename="interial_macros.xacro"/>
     <material name="white">
         <color rgba="1 1 1 1"/>
@@ -36,4 +37,7 @@
             </geometry>
         </collision>
+        <xacro:interial_box mass="0.5" x="0.26" y="0.2" z="0.06">
+            <origin xyz="0.13 0 0.03" rpy="0 0 0 "/>
+        </xacro:interial_box>
     </link>
     <!-- LEFT WHEEL LINK-->
@@ -56,4 +60,7 @@
             </geometry>
         </collision>
+        <xacro:inertial_cylinder mass="0.1" length="0.04" radius="0.05">
+            <origin xyz="0 0 0" rpy="0 0 0"/>
+        </xacro:inertial_cylinder>
     </link>
     <!-- RIGHT WHEEL LINK-->
@@ -76,4 +83,7 @@
             </geometry>
         </collision>
+        <xacro:inertial_cylinder mass="0.1" length="0.04" radius="0.05">
+            <origin xyz="0 0 0" rpy="0 0 0"/>
+        </xacro:inertial_cylinder>
     </link>
     <!-- FRONT WHEEL LINK-->
@@ -95,4 +105,7 @@
             </geometry>
         </collision>
+        <xacro:inertial_sphere mass="0.1" radius="0.05">
+            <origin xyz="0 0 0" rpy="0 0 0"/>
+        </xacro:inertial_sphere>
     </link>
 </robot>

Commit message: created lidar description, added 'red' as material

File: description/robot_core.xacro (robot description, xacro)
@@ -13,4 +13,7 @@
     <material name="black">
         <color rgba="0 0 0 1" />
+    </material>
+    <material name="red">
+        <color rgba="1 0 0 1"/>
     </material>
     <!-- BASE LINK -->

Commit message: changed position of back wheels from 0.175 to 0.1

File: description/robot_core.xacro (robot description, xacro)
@@ -40,5 +40,5 @@
                 <box size="0.26 0.2 0.06"/>
             </geometry>
-            <material name="white"/>
+            <material name="black"/>
         </visual>
         <collision>
@@ -56,5 +56,5 @@
         <parent link="base_link" />
         <child link="left_wheel"/>
-        <origin xyz="0 0.175 0" rpy="-${pi/2} 0 0"/>
+        <origin xyz="0 0.1 0" rpy="-${pi/2} 0 0"/>
         <axis xyz="0 0 1"/>
     </joint>
@@ -79,5 +79,5 @@
         <parent link="base_link" />
         <child link="right_wheel"/>
-        <origin xyz="0 -0.175 0" rpy="${pi/2} 0 0"/>
+        <origin xyz="0 -0.1 0" rpy="${pi/2} 0 0"/>
         <axis xyz="0 0 -1"/>
     </joint>
